File: PCB files/MainPCB/MainPCB.kicad_sch (KiCad schematic)
At the start: 153 parts, among them IC1 CYPD3177-24LQXQ, P1 Solder_Pad, P15 Solder_Pad, P16 Solder_Pad, P18 Solder_Pad, P19 Solder_Pad, P20 Solder_Pad, P21 Solder_Pad, P22 Solder_Pad, P25 Solder_Pad, P26 Solder_Pad, P27 Solder_Pad, P28 Solder_Pad, P29 Solder_Pad, P3 Solder_Pad, P30 Solder_Pad, P31 Solder_Pad, P32 Solder_Pad, P33 Solder_Pad, P34 Solder_Pad, P35 Solder_Pad, P4 Solder_Pad, P5 Solder_Pad, SW1 TS-1185EC-C-D-B, SW2 TS-1185EC-C-D-B, SW3 SK-3245S-L3-B, SW4 TS-1185EC-C-D-B, U1 SN74LVC1G373DBVR, U1 TPS53319DQPR, U10 MSM261D4030H1CPM, U11 AP40P05, U12 AO3400A, U13 SPX3819M5-L-3-3_TR, U14 SN74LVC2T45DCUR, U15 74LVC2G04DW-7, U16 X6511WR-03H-C30D60-R2, U17 X6511WR-03H-C30D60-R2, U18 X6511WR-03H-C30D60-R2, U19 X6511WR-03H-C30D60-R2, U2 TYPE-C-31-M-22, U21 X6511WR-06H-C30D60-R2, U22 X6511WR-06H-C30D60-R2, U23 ESP32-S3-WROOM-1, U24 SN74LVC2T45DCUR, U3 AO3401A, U4 AO3401A, U5 MS1040-R68M, U6 HSM4805, U9 SM4185T9RL

Commit message: update pcb design
Parts:
- removed C10, C11, C9: 100uF X5R, Capacitor_SMD:C_1206_3216Metric, symbol Device:C
- removed C11: 1nF, Capacitor_SMD:C_0402_1005Metric, symbol Device:C
- removed C11: Not used, Capacitor_SMD:C_0402_1005Metric, symbol Device:C
- removed C18, C31, C32, C33: 220uF, Capacitor_SMD:C_1206_3216Metric, symbol Device:C
- removed C20, C24: 10uF, Capacitor_SMD:C_0603_1608Metric, symbol Device:10uF 0603
- removed C22: 10nF, Capacitor_SMD:C_0402_1005Metric, symbol Device:10uF 0603
- removed C39: 0.1uF, Capacitor_SMD:C_0402_1005Metric, symbol Device:C
- removed JP7 (x6): SolderJumper_2_Open, Jumper:SolderJumper-2_P1.3mm_Open_RoundedPad1.0x1.5mm, symbol Jumper:SolderJumper_2_Open
- removed R10 (x2): 10K, Resistor_SMD:R_0603_1608Metric, symbol Device:R
- removed R11 (x2), R13: 1K, Resistor_SMD:R_0603_1608Metric, symbol Device:R
- removed R14: 49.9K, Resistor_SMD:R_0603_1608Metric, symbol Device:R
- removed R15: 100K, Resistor_SMD:R_0603_1608Metric, symbol Device:R
- removed R2: 220K, Resistor_SMD:R_0603_1608Metric, symbol Device:R
- removed R2: 47K, Resistor_SMD:R_0603_1608Metric, symbol Device:R
- removed R20, R23: 100K, Resistor_SMD:R_0603_1608Metric, symbol Device:10K 0603
- removed R25: 5.1K, Resistor_SMD:R_0603_1608Metric, symbol Device:R
- removed R3: Not used, Resistor_SMD:R_0603_1608Metric, symbol Device:R
- removed R3: 130K, Resistor_SMD:R_0603_1608Metric, symbol Device:R
- removed R3: 560K, Resistor_SMD:R_0603_1608Metric, symbol Device:R
- removed R3: 15K, Resistor_SMD:R_0603_1608Metric, symbol Device:R
- removed R3: 0, Resistor_SMD:R_0603_1608Metric, symbol Device:R
- removed TP1, TP2, TP3 (x9): TestPoint, TestPoint:TestPoint_Pad_D1.5mm, symbol Connector:TestPoint
- removed U11: AP40P05, footprint:SOT-23-3_L2.9-W1.3-P1.90-LS2.4-BR, symbol MyParts:AP40P05
- removed U13: SPX3819M5-L-3-3_TR, footprint:SOT-23-5_L3.0-W1.7-P0.95-LS2.8-BR, symbol MyParts:SPX3819M5-L-3-3_TR
- removed U3, U4: AO3401A, footprint:SOT-23_L2.9-W1.3-P1.90-LS2.4-BR, symbol MyParts:AO3401A
- removed U9: SM4185T9RL, footprint:TO-252-2_L6.6-W6.1-P4.57-LS10.1-BL-1, symbol MyParts:SM4185T9RL
- added C11: 1nF, Capacitor_SMD:C_0402_1005Metric, symbol Device:C
- added C14 (x3): 47uF, Capacitor_SMD:C_1206_3216Metric, symbol Device:C
- added C15: 10uF, Capacitor_SMD:C_0603_1608Metric, symbol Device:0.1uF 0603
- added R1, R15, R21, R5: 100K, Resistor_SMD:R_0603_1608Metric, symbol Device:10K 0603
- added R10: 10K, Resistor_SMD:R_0603_1608Metric, symbol Device:R
- added R11: 1K, Resistor_SMD:R_0603_1608Metric, symbol Device:R
- added R2: 51K, Resistor_SMD:R_0603_1608Metric, symbol Device:R
- added R2: 220K, Resistor_SMD:R_0603_1608Metric, symbol Device:R
- added R2: 20K, Resistor_SMD:R_0603_1608Metric, symbol Device:R
- added U3: LM2937IMP-3_3_NOPB, footprint:SOT-223_L6.5-W3.5-P2.30-LS7.0-BR, symbol MyParts:LM2937IMP-3_3_NOPB
- added U4, U8: AP40P05, footprint:SOT-23-3_L2.9-W1.3-P1.90-LS2.4-BR, symbol MyParts:AP40P05
- C15: value 22uF X5R -> 4.7uF; LCSC # C12891 -> C29823
- C8: value 100uF X5R -> 0.1uF; footprint Capacitor_SMD:C_1206_3216Metric -> Capacitor_SMD:C_0402_1005Metric; LCSC # C15008 -> C307331
- R1: footprint Resistor_SMD:R_0603_1608Metric -> Resistor_SMD:R_0402_1005Metric; LCSC # C22975 -> C4109
- R10: value 10K -> 5.1K; footprint Resistor_SMD:R_0603_1608Metric -> Resistor_SMD:R_0402_1005Metric; LCSC # C25804 -> C25905
- R15: value 100K -> 105K; LCSC # C25803 -> C325596
- R2: value 200K -> 105K; LCSC # C25811 -> C325596
- R25: footprint Resistor_SMD:R_0603_1608Metric -> Resistor_SMD:R_0402_1005Metric; LCSC # C22940 -> C25882
- R25: footprint Resistor_SMD:R_0603_1608Metric -> Resistor_SMD:R_0402_1005Metric; LCSC # C23186 -> C25905
- R3: value 47K -> 71.5K; LCSC # C25819 -> C228040
- R3: value 510K -> 150K; LCSC # C23192 -> C22807
- R3: value 3K -> 1.8K; LCSC # C4211 -> C4177
- R3: value 20K -> 10K; LCSC # C4184 -> C25804
- U23: value ESP32-S3-WROOM-1 -> ESP32-S3-WROOM-1-N8; LCSC # C2913197 -> C2913198
- U5: value MS1040-R68M -> MDA1050-2R2M; LCSC # C380043 -> C2847559
Connections:
- net 3.3V AFTER MOSFET is gone; now on net +3.3V: C14.2, C15.2, C23.2, C29.2, P34.1, U10.1 (VDD), U14.8 (VCCB), U24.8 (VCCB)
- net 5V AFTER MOSFET is gone; now on net +5V: C21.2, C28.2, P1.1, U14.1 (VCCA), U16.3, U17.3, U18.3, U19.3, U21.2, U21.4, U22.4, U22.6, U24.1 (VCCA)
- net STEPDOWN_ROVP is gone; now on net GND: U1.5 (ROVP)
- net STEPDOWN_VDC_IN is gone; now on net USB_PD_IC_VDC_OUT: C12.1, C13.1, C14.1, C15.1, C16.2, U1.12 (VIN), U1.13 (VIN), U1.14 (VIN), U1.15 (VIN), U1.16 (VIN), U1.17 (VIN), U1.19 (VDD)
- net +3.3V: now also C15.2, U3.3 (OUTPUT)
- net +5V: now also C35.2, R3.1, U5.1, C14.1, C14.1, C14.1, U4.3 (D), U8.3 (D)
- net GND: now also C8.1, SW3.1, C11.2, C14.2, C14.2, C14.2, C15.1, R1.2, R2.2, R2.2, U3.2 (GND), U3.4 (TAP); no longer C8.2
- net USB_PD_IC_FET_GATE: now also R10.1, R11.2
- net USB_PD_IC_VBUS_FET_EN: now also R11.1
- net USB_PD_IC_VDC_OUT: now also R15.2, R2.1, R21.2, R5.1, U4.2 (S), U8.2 (S)
- net VBUS: now also C8.2, R10.2, U3.1 (INPUT)
- net at U12.3 (D): now also R15.1, R21.1, U4.1 (G), U8.1 (G)
- net at U1.4 (VBST): now also C37.1
- net at R11.2: now also C11.1, R2.1, R2.2
- net IO10/VBUS to 5V LETCH: now reaches U23.18 (GPIO10/TOUCH10/ADC1_CH9/FSPICS0/FSPIIO4/SUBSPICS0)
- net IO10/VBUS to 5V LETCH: now also U1.1 (LE)
- net IO7/USB PD VOLTS DETECTION: now reaches U23.7 (GPIO7/TOUCH7/ADC1_CH6)
- net IO7/USB PD VOLTS DETECTION: now also R2.1, R5.2
- net IO15/LED LETCH EN: no longer names the net of U23.8 (GPIO15/U0RTS/ADC2_CH4/XTAL_32K_P)
- net IO15/LED LETCH EN: no longer U1.1 (LE)
- net IO16/POWERMOSFETS: no longer names the net of U23.9 (GPIO16/U0CTS/ADC2_CH5/XTAL_32K_N)
- net IO16/POWERMOSFETS: no longer U1.3 (D)
- net IO2/USB PD FAULT renamed IO2/VBUS TO 5V MOSFET
- net IO2/VBUS TO 5V MOSFET: now also U1.3 (D); no longer IC1.9 (FAULT)
- net IO6/MODE DETECTION renamed IO6/USB PD AMPS DETECTION
- net STEPDOWN_RF: no longer names the net of U1.22 (RF)
- removed net STEPDOWN_VDC_OUT: C35.2, C8.1, R3.1, U5.1
- net USB_PD_IC_SAFE_PWR_EN: no longer names the net of IC1.4 (SAFE_PWR_EN)
- new net USB_PD_IC_FAULT: IC1.9 (FAULT), R1.1
- no-connect marks 26 -> 24
Other:
- note added: "GlowLight (5V)"
- note added: "GlowTower (3A)"
- note added: "Stepdown converter will only turn on if USB_PD_IC_VDC_OUT is 9V or higher."
- note added: "TI webench: 3x 22uF + 1x 4.7uF, not 4x 22uF"
- note added: "TI webench: 3x 47uF, not 4x 100uF"
- note added: "USB-C PD to 5V"
- note added: "VBUS to 5V"
- note removed: "Default: 500khz RF"
- note removed: "GlowLight (9V)"
- note removed: "GlowTower (4A)"
- note removed: "LED power"
- note removed: "Not very clear yet what voltage divider to use to get 5V. My calculations said for example 20K and 134K. But a user online used 20K and 47K. Plan: test multiple resistor values with first ordered PCB and see which gives out 5V."
- note removed: "Power need: GlowLight: (((0,055A*60)+0,3A)*5V)*80% efficiency = 22W total power requirement from power supply -> VBUS MIN 9V, ISNK_COARSE 2A, ISNK_FINE +500 (required: 25W power supply, starting at 8 EUR) GlowTower: (((0,055A*240)+0,3A)*5V)* 80% efficiency = 81W total power requirement from power source -> VBUS MIN 20V, ISNK_COARSE 4A, ISNK_FINE +500 (required: 100W power supply, starting at 26 E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"
- note removed: "Step down"
- note removed: "Testing procedure once I receive PCB prototype: Step 1: test USB-C PD IC only: - does 9V output work? - does 20V output work? - does 5V output work for devices which don't support 9V or 20V? Step 2: connect step down (EN and VIN) and test step down: - does it output 5V? - is the voltage stable? how about noise? Step 3: connect step down output to 5V and test whole system: - 5v stable? for low and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"
- note removed: "V TRIP: 5.6V (560K resistor) or 5.1V (510K resistor Note: 510K is basic component and therefore cheaper, but might be to close to target voltage"
- moved on the sheet: C16, C17, C19, R1, R10, R11, R19, R2, R25, R3, U1, U12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

Commit message: added pinout for main pcb 2.0 and new photos
Parts:
- removed C15: 10uF, Capacitor_SMD:C_0603_1608Metric, symbol Device:0.1uF 0603
- removed C8: 0.1uF, Capacitor_SMD:C_0402_1005Metric, symbol Device:C
- removed R25: 2.4K, Resistor_SMD:R_0402_1005Metric, symbol Device:R
- removed R25: 5.1K, Resistor_SMD:R_0402_1005Metric, symbol Device:R
- removed U3: LM2937IMP-3_3_NOPB, footprint:SOT-223_L6.5-W3.5-P2.30-LS7.0-BR, symbol MyParts:LM2937IMP-3_3_NOPB
- added C1, C2: 0.1uF, Capacitor_SMD:C_0402_1005Metric, symbol Device:C
- added C3: 33nF, Capacitor_SMD:C_0603_1608Metric, symbol Device:C
- added C4: 10uF, Capacitor_SMD:C_0805_2012Metric, symbol Device:C
- added C5: 47pF, Capacitor_SMD:C_0402_1005Metric, symbol Device:C
- added C6: 47uF, Capacitor_SMD:C_0805_2012Metric, symbol Device:C
- added L1: CPY201209T-4R7M-NP, footprint:L0805, symbol MyParts:CPY201209T-4R7M-NP
- added R1: 30.9K, Resistor_SMD:R_0402_1005Metric, symbol Device:R
- added R2: 10K, Resistor_SMD:R_0402_1005Metric, symbol Device:R
- added U1: TPS62933DRLR, footprint:SOT-583-8_L2.1-W1.2-P0.50-LS1.6-BR, symbol MyParts:TPS62933DRLR
Connections:
- net USB_PD_IC_ISNK_FINE is gone; now on net GND: IC1.6 (ISNK_FINE)
- net +3.3V: now also C5.2, C6.2, L1.2, R1.1
- net GND: now also C2.1, C3.1, C4.1, C6.1, R2.2, U1.4 (GND)
- net VBUS: now also C2.2, C4.2, U1.3 (VIN)
- new net: C5.1, R1.2, R2.1, U1.8 (FB)
- new net: C1.2, L1.1, U1.5 (SW)
- new net: C1.1, U1.6 (BST)
- new net: C3.2, U1.7 (SS)
Other:
- note added: "Designed for VIN 4.8V to 21V, at 1A max output. Based on webench.ti.com."
- note added: "FINE SETTING +0"
- note added: "USB-C PD to 3.3V"
- note removed: "3.3V converter"
- note removed: "FINE SETTING +500"
- note removed: "Info: The 5-V LDO is not controlled by the EN pin. The LDO starts-up any time VDD rises to approximately 2 V."
- note removed: "TI webench: 3x 22uF + 1x 4.7uF, not 4x 22uF"
- note removed: "TI webench: 3x 47uF, not 4x 100uF"
- note removed: "TODO: - calculate R1 and R2 (in datasheet), to set output voltage - calculate inductor formulas - calculate output capacitors - calculate R TRIP overcurrent resistor - 9.2.2.2.2 Redundant Overvoltage Protection (datasheet) Question: - do I need separate resistor pairs for both 9V and 20V input?"
- note removed: "Warning: internal LDO is 5V, so pins likely need voltage divider to be connected to esp32"
- moved on the sheet: C11, C12, C13, C14, C15, C16, C17, C35, C37, R11, R15, R2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

Commit message: added new documents
Other:
- note added: "!!! Redesign plan !!!"
- note added: "Switching from one buck/boost to four buck/boost, using TPS55289 (can output everything from 0.8V to 22V, even selectable via I2C! perfect for LEDs) Would optimize for 12V leds, but can always switch back to 5V without hardware change needed (except maybe problems with inductor?)"
Changed lines of the file:
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@@
     (effects (font (size 3 3)) (justify left bottom))
+  )
+  (text "Switching from one buck/boost to four buck/boost, using TPS55289\n(can output everything from 0.8V to 22V, even selectable via I2C! \nperfect for LEDs)\nWould optimize for 12V leds, but can always switch back to 5V\nwithout hardware change needed (except maybe problems with inductor?)"
+    (at 300.355 260.35 0)
+    (effects (font (size 2 2)) (justify left bottom))
   )
   (text "VBUS MAX 20V" (at 225.425 150.495 0)
@@
     (effects (font (size 3 3)) (justify left bottom))
   )
+  (text "!!! Redesign plan !!!" (at 300.99 238.76 0)
+    (effects (font (size 3 3)) (justify left bottom))
+  )
